File: hw/analog-phone-interface-module/analog-phone-interface-module.kicad_sch (KiCad schematic)
At the start: 7 parts, among them J1 Screw_Terminal_01x03, J2 Screw_Terminal_01x06, J3 Screw_Terminal_01x04, J4 Screw_Terminal_01x04, J5 8P8C_Shielded, J6 Screw_Terminal_01x03, J7 RJ11_Shielded

Commit message: Small update to schematic
Parts:
- removed J3: Screw_Terminal_01x04, symbol Connector:Screw_Terminal_01x04
- added J3: Screw_Terminal_01x06, symbol Connector:Screw_Terminal_01x06
Connections:
- net +12V: now also J3.2 (Pin_2)
- net -12V: now also J3.3 (Pin_3)
- net -48V: now also J3.5 (Pin_5)
- net GND: now also J3.4 (Pin_4)
- new net +5V: J3.1 (Pin_1)
- new net GND1: J3.6 (Pin_6)
Other:
- sheet Phone line interface circuit ports: added ring-voltage-n, ring-voltage-p; removed none
- note added: "Real PSTN uses -48V, but -12V is sufficient here. Just bridge the -48V and -12V terminal externally"
- note removed: "12V DC power supply Real PSTN uses -48V, but -12V is sufficient here. Just bridge the -48V and -12V terminal externally"
