File: hw/analog-phone-interface-module/phone-line-interface-circuit.kicad_sch (KiCad schematic)
At the start: 4 parts, among them U1 74AUC1G66, U2 4N35, U4 4016

Commit message: Small update to schematic
Parts:
- removed U1: 74AUC1G66, symbol 74xGxx:74AUC1G66
- removed U4: 4016, symbol 4xxx:4016
- added C5: 4u, symbol Device:C
- added C6: 100n, symbol Device:C
- added D1: D, symbol Device:D
- added R10, R11, R9: 330R, symbol Device:R
- added R12, R7: R, symbol Device:R
- added R8: 600R, symbol Device:R
- added U1, U4, U5: MOC3020M, symbol Relay_SolidState:MOC3020M
- added U6: 74HCT00, symbol 74xx:74HCT00
Connections:
- net line-enable: now also U6.1, U6.10, U6.2, U6.9
- net off-hook-signal: now also U6.11
- net phone-line-tip: now also C5.2, D1.2 (A), U1.4
- net ring-voltage-enable: now also R11.1
- net to-pbx-matrix: now also U5.6
- net at L2.2, U2.1: now also D1.1 (K)
- net GND: now reaches U2.4
- net GND: now also C6.2, U1.2, U4.2, U5.2, U6.7 (GND)
- net at U2.5: now also R12.2, U6.12, U6.13
- net at L2.1: now also R7.2
- new net: R11.2, U1.1
- new net: R8.2, U4.6
- new net: C5.1, U4.4, U5.4
- new net: R9.2, U5.1
- new net: R10.2, U4.1
- new net: R10.1, U6.6
- new net: U6.3, U6.4, U6.5
- new net: R9.1, U6.8
- new net +5V: C6.1, R12.1, U6.14 (VCC)
- new net -48V: R7.1
- new net GND1: R8.1
- new net ring-voltage-p: U1.6
Other:
- moved on the sheet: L2, U2
